Commit message: Implement 61529d3: Improve stability of the simulation pkg

File: racecar_description/urdf/macros.xacro (robot description, xacro)
@@ -41,5 +41,5 @@
   <origin xyz="0 0 0.05" rpy="0 0 0" />
   <geometry>
-    <mesh filename="package://racecar_description/meshes/chassis.STL" />
+    <mesh filename="file://$(find racecar_description)/meshes/chassis.STL" />
   </geometry>
 </xacro:macro>
@@ -47,5 +47,5 @@
   <origin xyz="0 0 0" rpy="0 0 0" />
   <geometry>
-    <mesh filename="package://racecar_description/meshes/left_rear_wheel.STL" />
+    <mesh filename="file://$(find racecar_description)/meshes/left_rear_wheel.STL" />
   </geometry>
 </xacro:macro>
@@ -53,5 +53,5 @@
   <origin xyz="0 0 0" rpy="0 0 0" />
   <geometry>
-    <mesh filename="package://racecar_description/meshes/right_rear_wheel.STL" />
+    <mesh filename="file://$(find racecar_description)/meshes/right_rear_wheel.STL" />
   </geometry>
 </xacro:macro>
@@ -59,5 +59,5 @@
   <origin xyz="0 0 0" rpy="0 0 0" />
   <geometry>
-    <mesh filename="package://racecar_description/meshes/left_front_wheel.STL" />
+    <mesh filename="file://$(find racecar_description)/meshes/left_front_wheel.STL" />
   </geometry>
 </xacro:macro>
@@ -65,5 +65,5 @@
   <origin xyz="0 0 0" rpy="0 0 0" />
   <geometry>
-    <mesh filename="package://racecar_description/meshes/right_front_wheel.STL" />
+    <mesh filename="file://$(find racecar_description)/meshes/right_front_wheel.STL" />
   </geometry>
 </xacro:macro>
@@ -71,5 +71,5 @@
   <origin xyz="0 0 0" rpy="0 0 0" />
   <geometry>
-    <mesh filename="package://racecar_description/meshes/left_steering_hinge.STL" />
+    <mesh filename="file://$(find racecar_description)/meshes/left_steering_hinge.STL" />
   </geometry>
 </xacro:macro>
@@ -77,5 +77,5 @@
   <origin xyz="0 0 0" rpy="0 0 0" />
   <geometry>
-    <mesh filename="package://racecar_description/meshes/right_steering_hinge.STL" />
+    <mesh filename="file://$(find racecar_description)/meshes/right_steering_hinge.STL" />
   </geometry>
 </xacro:macro>

File: racecar_description/urdf/racecar.xacro (robot description, xacro)
@@ -173,5 +173,5 @@
       <origin xyz="0 0 0" rpy="0 0 0"/>
       <geometry>
-        <mesh filename="package://racecar_description/meshes/hokuyo.dae"/>
+        <mesh filename="file://$(find racecar_description)/meshes/hokuyo.dae"/>
         <material name="DarkGrey" />
       </geometry>
